File: V0/Design/HW.ACIM-PSU/Power_Supply.kicad_sch (KiCad schematic)
At the start: 91 parts, among them J1 AC POWER INPUT, M1 470V/1.2kA, M2 470V/1.2kA, M3 470V/1.2kA, M4 470V/1.2kA, Q1 20V/1A, Q2 20V/1A, U1 Buck 5V/1.5A, U2 LDO 3.3V/1.5A, U3 LDO 3.3V/20mA

Commit message: V0 production files update 2
Parts:
- C20, C21, C22, C23, C24, C25, C26, C27, C29, C30, C31, C33, C34, D2, D3, FT4, Q1, R10, R11, R12, RL1, U2, U3: now not fitted
Changed lines of the file:
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@@
 		)
 	)
+	(text_box "Use R0 instead of diode for D4"
+		(exclude_from_sim no)
+		(at 180.34 81.915 0)
+		(size 22.86 5.08)
+		(stroke
+			(width -0.0001)
+			(type default)
+			(color 200 0 0 1)
+		)
+		(fill
+			(type none)
+		)
+		(effects
+			(font
+				(size 1.27 1.27)
+				(color 200 0 0 1)
+			)
+			(justify top)
+		)
+	)
+	(text_box "Short circuit pin 5 & 6 of RL1"
+		(exclude_from_sim no)
+		(at 170.815 46.99 0)
+		(size 17.78 5.08)
+		(stroke
+			(width -0.0001)
+			(type default)
+			(color 200 0 0 1)
+		)
+		(fill
+			(type none)
+		)
+		(effects
+			(font
+				(size 1.27 1.27)
+				(color 200 0 0 1)
+			)
+			(justify top)
+		)
+	)
 	(hierarchical_label "RL_INRUSH_EN"
 		(shape input)
@@
 		(in_bom yes)
 		(on_board yes)
-		(dnp no)
+		(dnp yes)
 		(fields_autoplaced yes)
 		(property "Reference" "C33"
@@
 		(in_bom yes)
 		(on_board yes)
-		(dnp no)
+		(dnp yes)
 		(property "Reference" "C24"
 			(at 217.805 137.1599 90)
@@
 		(in_bom yes)
 		(on_board yes)
-		(dnp no)
+		(dnp yes)
 		(property "Reference" "R11"
 			(at 135.89 66.04 0)
@@
 		(in_bom yes)
 		(on_board yes)
-		(dnp no)
+		(dnp yes)
 		(fields_autoplaced yes)
 		(property "Reference" "C22"
@@
 		(in_bom yes)
 		(on_board yes)
-		(dnp no)
+		(dnp yes)
 		(property "Reference" "C21"
 			(at 160.02 36.195 0)
@@
 		(in_bom yes)
 		(on_board yes)
-		(dnp no)
+		(dnp yes)
 		(property "Reference" "C26"
 			(at 238.125 106.6799 90)
@@
 		(in_bom yes)
 		(on_board yes)
-		(dnp no)
+		(dnp yes)
 		(fields_autoplaced yes)
 		(property "Reference" "C27"
@@
 		(in_bom yes)
 		(on_board yes)
-		(dnp no)
+		(dnp yes)
 		(property "Reference" "Q1"
 			(at 136.525 57.15 90)
@@
 		(in_bom yes)
 		(on_board yes)
-		(dnp no)
+		(dnp yes)
 		(property "Reference" "C23"
 			(at 202.565 106.6799 90)
@@
 		(in_bom yes)
 		(on_board yes)
-		(dnp no)
+		(dnp yes)
 		(fields_autoplaced yes)
 		(property "Reference" "C31"
@@
 		(in_bom yes)
 		(on_board yes)
-		(dnp no)
+		(dnp yes)
 		(property "Reference" "RL1"
 			(at 158.75 46.99 0)
@@
 		(in_bom yes)
 		(on_board yes)
-		(dnp no)
+		(dnp yes)
 		(property "Reference" "U3"
 			(at 217.805 96.52 0)
@@
 		(in_bom yes)
 		(on_board yes)
-		(dnp no)
+		(dnp yes)
 		(property "Reference" "D2"
 			(at 146.05 74.93 0)
@@
 		(in_bom yes)
 		(on_board yes)
-		(dnp no)
+		(dnp yes)
 		(fields_autoplaced yes)
 		(property "Reference" "C30"
@@
 		(in_bom yes)
 		(on_board yes)
-		(dnp no)
+		(dnp yes)
 		(fields_autoplaced yes)
 		(property "Reference" "C34"
@@
 		(in_bom yes)
 		(on_board yes)
-		(dnp no)
+		(dnp yes)
 		(property "Reference" "R10"
 			(at 135.89 74.93 0)
@@
 		(in_bom yes)
 		(on_board yes)
-		(dnp no)
+		(dnp yes)
 		(property "Reference" "C20"
 			(at 183.515 132.0799 90)
@@
 		(in_bom yes)
 		(on_board yes)
-		(dnp no)
+		(dnp yes)
 		(property "Reference" "U2"
 			(at 200.025 123.19 0)
@@
 		(in_bom yes)
 		(on_board yes)
-		(dnp no)
+		(dnp yes)
 		(property "Reference" "R12"
 			(at 181.61 74.93 0)
@@
 		(in_bom yes)
 		(on_board yes)
-		(dnp no)
+		(dnp yes)
 		(property "Reference" "C25"
 			(at 227.965 132.0799 90)
@@
 		(in_bom yes)
 		(on_board yes)
-		(dnp no)
+		(dnp yes)
 		(fields_autoplaced yes)
 		(property "Reference" "FT4"
@@
 		(in_bom yes)
 		(on_board yes)
-		(dnp no)
+		(dnp yes)
 		(fields_autoplaced yes)
 		(property "Reference" "C29"
@@
 		(in_bom yes)
 		(on_board yes)
-		(dnp no)
+		(dnp yes)
 		(property "Reference" "D3"
 			(at 158.75 66.04 0)
