File: Design/HW.ACIM-PSU/MCUPOWER.kicad_sch (KiCad schematic)
At the start: 29 parts, among them J5 FAN, J6 MCU PWR, U3 SMPS 12V±2%/0.8A, U4 LDO 5V±1%, U5 LDO 3V3±2%

Commit message: V1 layout
Connections:
- net at C19.1, FT4.2: now also MD2.2 (ACL); no longer MD2.1 (ACN)
- net at C19.2, FT4.4: now also MD2.1 (ACN); no longer MD2.2 (ACL)
Changed lines of the file:
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@@
 	)
 	(junction
-		(at 59.69 57.15)
+		(at 38.1 31.75)
 		(diameter 0)
 		(color 0 0 0 0)
 	)
 	(junction
-		(at 81.28 31.75)
+		(at 59.69 57.15)
 		(diameter 0)
 		(color 0 0 0 0)
 	)
 	(junction
-		(at 153.67 57.15)
+		(at 81.28 31.75)
 		(diameter 0)
 		(color 0 0 0 0)
 	)
 	(junction
-		(at 60.96 21.59)
+		(at 153.67 57.15)
 		(diameter 0)
 		(color 0 0 0 0)
 	)
 	(junction
-		(at 38.1 21.59)
+		(at 60.96 21.59)
 		(diameter 0)
 		(color 0 0 0 0)
@@
 	)
 	(junction
-		(at 38.1 31.75)
-		(diameter 0)
-		(color 0 0 0 0)
-	)
-	(junction
 		(at 60.96 31.75)
 		(diameter 0)
@@
 	)
 	(junction
+		(at 38.1 21.59)
+		(diameter 0)
+		(color 0 0 0 0)
+	)
+	(junction
 		(at 123.825 57.15)
 		(diameter 0)
@@
 	(wire
 		(pts
-			(xy 35.56 31.75) (xy 38.1 31.75)
+			(xy 35.56 21.59) (xy 38.1 21.59)
 		)
 		(stroke
@@
 	(wire
 		(pts
+			(xy 38.1 21.59) (xy 41.91 21.59)
+		)
+		(stroke
+			(width 0.254)
+			(type default)
+		)
+	)
+	(wire
+		(pts
 			(xy 81.28 20.32) (xy 81.28 21.59)
 		)
@@
 	(wire
 		(pts
-			(xy 38.1 22.86) (xy 38.1 21.59)
+			(xy 38.1 30.48) (xy 38.1 31.75)
 		)
 		(stroke
@@
 	(wire
 		(pts
-			(xy 38.1 21.59) (xy 41.91 21.59)
-		)
-		(stroke
-			(width 0.254)
-			(type default)
-		)
-	)
-	(wire
-		(pts
 			(xy 134.62 62.23) (xy 134.62 66.04)
 		)
@@
 	(wire
 		(pts
-			(xy 35.56 21.59) (xy 38.1 21.59)
+			(xy 35.56 31.75) (xy 38.1 31.75)
 		)
 		(stroke
@@
 	(wire
 		(pts
-			(xy 38.1 31.75) (xy 41.91 31.75)
+			(xy 59.69 72.39) (xy 58.42 72.39)
 		)
 		(stroke
@@
 	(wire
 		(pts
-			(xy 59.69 72.39) (xy 58.42 72.39)
+			(xy 60.96 31.75) (xy 57.15 31.75)
 		)
 		(stroke
@@
 	(wire
 		(pts
-			(xy 60.96 31.75) (xy 57.15 31.75)
+			(xy 165.1 88.9) (xy 154.94 88.9)
 		)
 		(stroke
@@
 	(wire
 		(pts
-			(xy 165.1 88.9) (xy 154.94 88.9)
+			(xy 38.1 31.75) (xy 41.91 31.75)
 		)
 		(stroke
@@
 	(wire
 		(pts
-			(xy 38.1 31.75) (xy 38.1 30.48)
+			(xy 38.1 21.59) (xy 38.1 22.86)
 		)
 		(stroke
@@
 	(symbol
 		(lib_id "SAMPI:CERCAP")
-		(at 35.56 27.94 90)
+		(at 35.56 25.4 90)
+		(mirror x)
 		(unit 1)
 		(exclude_from_sim no)
@@
 		)
 		(property "Value" "100nF/400V"
-			(at 40.64 22.86 0)
+			(at 40.64 30.48 0)
 			(effects
 				(font
@@
 		)
 		(property "Footprint" "SAMPI:CAP_FILM_6.0x12.0x12.5-P10"
-			(at 35.56 27.94 0)
+			(at 35.56 25.4 0)
 			(effects
 				(font
@@
 		)
 		(property "Datasheet" ""
-			(at 35.56 27.94 0)
+			(at 35.56 25.4 0)
 			(effects
 				(font
@@
 		)
 		(property "Description" "CAP FILM 0.1UF 20% 560VDC RADIAL"
-			(at 35.56 27.94 0)
+			(at 35.56 25.4 0)
 			(effects
 				(font
@@
 		)
 		(property "MNP" "BFC233824104"
-			(at 35.56 27.94 90)
+			(at 35.56 25.4 90)
 			(effects
 				(font
@@
 		)
 		(property "MFT" "VISHAY"
-			(at 35.56 27.94 0)
+			(at 35.56 25.4 0)
 			(effects
 				(font
@@
 	(symbol
 		(lib_id "SAMPI:AC2")
-		(at 27.94 31.75 90)
-		(mirror x)
+		(at 27.94 21.59 90)
 		(unit 1)
 		(exclude_from_sim no)
@@
 		(dnp no)
 		(property "Reference" "#PWR043"
-			(at 31.75 31.75 0)
+			(at 31.75 21.59 0)
 			(effects
 				(font
@@
 		)
 		(property "Value" "AC2"
-			(at 22.86 31.75 90)
+			(at 22.86 21.59 90)
 			(effects
 				(font
@@
 		)
 		(property "Footprint" ""
-			(at 27.94 31.75 0)
+			(at 27.94 21.59 0)
 			(effects
 				(font
@@
 		)
 		(property "Datasheet" ""
-			(at 27.94 31.75 0)
+			(at 27.94 21.59 0)
 			(effects
 				(font
@@
 		)
 		(property "Description" ""
-			(at 27.94 31.75 0)
+			(at 27.94 21.59 0)
 			(effects
 				(font
@@
 	(symbol
 		(lib_id "SAMPI:AC1")
-		(at 27.94 21.59 90)
+		(at 27.94 31.75 90)
+		(mirror x)
 		(unit 1)
 		(exclude_from_sim no)
@@
 		(dnp no)
 		(property "Reference" "#PWR042"
-			(at 31.75 21.59 0)
+			(at 31.75 31.75 0)
 			(effects
 				(font
@@
 		)
 		(property "Value" "AC1"
-			(at 22.86 21.59 90)
+			(at 22.86 31.75 90)
 			(effects
 				(font
@@
 		)
 		(property "Footprint" ""
-			(at 27.94 21.59 0)
+			(at 27.94 31.75 0)
 			(effects
 				(font
@@
 		)
 		(property "Datasheet" ""
-			(at 27.94 21.59 0)
+			(at 27.94 31.75 0)
 			(effects
 				(font
@@
 		)
 		(property "Description" ""
-			(at 27.94 21.59 0)
+			(at 27.94 31.75 0)
 			(effects
 				(font
@@
 	(symbol
 		(lib_id "SAMPI:CK_Choke_2")
-		(at 29.845 35.56 0)
-		(mirror x)
+		(at 29.845 17.78 0)
 		(unit 1)
 		(exclude_from_sim no)
@@
 		(dnp no)
 		(property "Reference" "FT4"
-			(at 31.115 16.51 0)
+			(at 31.75 17.145 0)
 			(effects
 				(font
@@
 		)
 		(property "Value" "15mH/500mA"
-			(at 31.115 19.05 0)
+			(at 31.75 19.05 0)
 			(effects
 				(font
@@
 		)
 		(property "Footprint" "SAMPI:EE8.3"
-			(at 29.845 35.56 0)
+			(at 29.845 17.78 0)
 			(effects
 				(font
@@
 		)
 		(property "Datasheet" ""
-			(at 29.845 35.56 0)
+			(at 29.845 17.78 0)
 			(effects
 				(font
@@
 		)
 		(property "Description" "15MH 2 LINE COMMON MODE CHOKE TH"
-			(at 29.845 35.56 0)
+			(at 29.845 17.78 0)
 			(effects
 				(font
@@
 		)
 		(property "MNP" "EE8.3-15MH"
-			(at 31.75 34.29 0)
+			(at 31.75 19.05 0)
 			(effects
 				(font
@@
 		)
 		(property "MFT" "OEM"
-			(at 29.845 35.56 0)
+			(at 29.845 17.78 0)
 			(effects
 				(font

Commit message: V1 layout update 1
Parts:
- removed D7: PWR, SAMPI:LED0603, symbol SAMPI:WLED
- removed R15: 1K, SAMPI:RES0603, symbol SAMPI:RES
