File: Design/HW.ACIM-PSU/HW.ACIM-PSU.kicad_pcb (KiCad board)
At the start: 4 copper layers, 98 x 98 mm, 90 parts, among them J2 LINE, J3 INV PWR & RELAYS, J4 HIGH VOLTAGE OUTPUTS, J5 FAN, J6 MCU PWR, J7 TE, J8 NEUTRAL, M1 470V/1.2kA, M2 470V/1.2kA, M3 470V/1.2kA, Q1 20V/1A, Q2 20V/1A, U1 SMPS 16V±2%/0.6A, U2 LDO 5V±1%, U3 SMPS 12V±2%/0.8A, U4 LDO 5V±1%, U5 LDO 3V3±2%

Commit message: V1 layout
Parts:
- C21, C4, D1, D2, D3, D4, D5, D6, Q1, Q2, R10, R11: moved to B.Cu
- moved C4 189.0 mm to (87.1, 141.6), turned to 180 degrees
- moved D1 188.5 mm to (87.1, 144.6), turned to 180 degrees
- moved D2 180.8 mm to (121.6, 135.4)
- moved D5 177.1 mm to (121.7, 131.9), turned to 180 degrees
- moved D3 175.2 mm to (130.8, 131.7), turned to 180 degrees
- moved D4 175.2 mm to (130.8, 134.8), turned to 180 degrees
- moved R10 150.3 mm to (135.1, 134.8), turned to 180 degrees
- moved R11 146.7 mm to (135.3, 130.8), turned to 180 degrees
- moved Q1 146.1 mm to (127.7, 140.0), turned to 180 degrees
- moved Q2 144.2 mm to (133.7, 138.5), turned to 180 degrees
- moved C1 135.4 mm to (103.1, 140.2), turned to -90 degrees
- moved D6 88.0 mm to (151.6, 144.6), turned to 180 degrees
- moved C23 83.4 mm to (132.4, 139.6), turned to -90 degrees
- moved C21 73.4 mm to (151.6, 141.6), turned to 180 degrees
- moved C19 67.6 mm to (104.3, 105.8), turned to -90 degrees
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Connections:
- C19 pad 1: Net-(MD2-ACN) -> Net-(MD2-ACL)
- C19 pad 2: Net-(MD2-ACL) -> Net-(MD2-ACN)
- C6 pad 1: Net-(MD1-ACN) -> Net-(MD1-ACL)
- C6 pad 2: Net-(MD1-ACL) -> Net-(MD1-ACN)
- FT1 pad 2: Net-(MD1-ACL) -> Net-(MD1-ACN)
- FT1 pad 4: Net-(MD1-ACN) -> Net-(MD1-ACL)
- FT4 pad 2: Net-(MD2-ACN) -> Net-(MD2-ACL)
- FT4 pad 4: Net-(MD2-ACL) -> Net-(MD2-ACN)
- J4 pad 10: VDC -> PGND
- J4 pad 4: PGND -> VDC
- J4 pad 5: PGND -> VDC
- J4 pad 6: PGND -> VDC
- J4 pad 8: VDC -> PGND
- J4 pad 9: VDC -> PGND
Routing:
- net Net-(MD2-ACN): track 0.00 -> 60.5 mm
- net Net-(MD2-ACL): track 0.00 -> 51.2 mm
- net +24V_INV: track 0.00 -> 36.3 mm
- net Net-(MD1-ACL): track 0.00 -> 27.5 mm
- net VDC: track 37.5 -> 62.3 mm
- net Net-(RL2-NC): track 120.1 -> 142.1 mm
- net PGND: track 102.9 -> 121.8 mm
- net GND_INV: track 0.00 -> 17.2 mm
- net Net-(MD1-ACN): track 0.00 -> 13.4 mm
- net AC1: track 46.3 -> 40.3 mm
- net Net-(BR1-DC+): track 16.8 -> 21.7 mm
- net AC2: track 31.2 -> 33.6 mm
Other:
- outline, holes or cut-outs redrawn

Commit message: V1 layout update 1
Parts:
- added C31: 10uF/35V, SAMPI:CAP1206, B.Cu at (163.7, 104.1)
- added SH9: SCREW HOLDER, SAMPI:SCREWHOLE-2.5M, F.Cu at (110.1, 138.2)
- C10: value 470uF/25V -> 220uF/25V; footprint SAMPI:CAP_ELEC-10.3x10.3-DIA10 -> SAMPI:CAP_ELEC-8.3x8.3-DIA8.0
- C12, C17, C18, C2, C20, C22, C25, C26, C27, C28, C29, C3, C30, C5, C7, L1, L2, R1, R12, R13, R14, R2, R3, U1, U2, U3, U4, U5: moved to B.Cu
- moved U1 223.4 mm to (76.6, 137.5), turned to 180 degrees
- moved L1 206.8 mm to (76.6, 128.3), turned to 90 degrees
- moved R3 203.9 mm to (79.0, 141.2), turned to 90 degrees
- moved R1 201.2 mm to (75.8, 141.2), turned to -90 degrees
- moved C3 198.7 mm to (77.4, 141.2), turned to 90 degrees
- moved R2 195.8 mm to (79.0, 137.5), turned to 90 degrees
- moved C5 194.4 mm to (76.6, 134.4)
- moved C7 185.2 mm to (81.7, 124.9), turned to 90 degrees
- moved C2 183.9 mm to (73.9, 137.5), turned to -90 degrees
- moved C10 152.7 mm to (78.2, 124.2), turned to 180 degrees
- moved J5 129.4 mm to (112.3, 144.5), turned to 180 degrees
- moved U2 121.4 mm to (164.5, 107.7), turned to 90 degrees
- moved C12 112.4 mm to (162.9, 111.1)
- moved U3 109.1 mm to (134.2, 137.8), turned to -90 degrees
- moved C24 108.9 mm to (121.5, 141.3), turned to 90 degrees
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Connections:
- D4 pad K: Net-(RL2-COIL1) -> Net-(RL2-COIL2)
- D5 pad A: Net-(RL2-COIL1) -> Net-(RL2-COIL2)
- D7 pad A: Net-(D7-PadA) -> +5V_INV
- D7 pad K: GND_MCU -> Net-(D7-PadK)
- J3 pad 7: /INVERTER POWER/~{DEV_RELAY} -> /INVERTER POWER/PWR_RELAY
- J3 pad 8: /INVERTER POWER/PWR_RELAY -> /INVERTER POWER/~{DEV_RELAY}
- R15 pad 1: +3V3_MCU -> Net-(D7-PadK)
- R15 pad 2: Net-(D7-PadA) -> GND_INV
- RL2 pad 1: Net-(RL2-COIL1) -> +12V_MCU
- RL2 pad 2: +12V_MCU -> Net-(RL2-COIL2)
Routing:
- net GND_MCU: track 0.00 -> 223.3 mm
- net GND_INV: track 17.2 -> 211.0 mm
- net +12V_MCU: track 0.00 -> 188.9 mm, vias 0 -> 7
- net +16V_INV: track 0.00 -> 126.1 mm, vias 0 -> 3
- net Net-(RL2-COIL2): track 0.00 -> 98.3 mm, vias 0 -> 2
- net Net-(RL1-COIL1): track 0.00 -> 61.8 mm, vias 0 -> 2
- net +24V_MCU: track 0.00 -> 53.5 mm
- net PGND: track 121.8 -> 173.6 mm
- net +5V_INV: track 0.00 -> 23.2 mm
- net +3V3_MCU: track 0.00 -> 17.1 mm
- net Net-(MD1-ACN): track 13.4 -> 23.9 mm
- net +5V_MCU: track 0.00 -> 8.49 mm
- net Net-(U3-SW): track 0.00 -> 7.25 mm
- net Net-(MD1-ACL): track 27.5 -> 33.9 mm
- net Net-(U1-VFB): track 0.00 -> 4.90 mm
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
Commit message: V1 layout update 2
Routing:
- net Net-(RL1-COIL1): track 61.8 -> 74.5 mm
- net Net-(RL2-COIL2): track 98.3 -> 109.9 mm
- net +12V_MCU: track 188.9 -> 200.4 mm
Other:
- outline, holes or cut-outs redrawn

Commit message: V1 layout update 3
Routing:
- net GND_MCU: track 223.3 -> 7.30 mm, vias 0 -> 13
- net GND_INV: track 211.0 -> 0.00 mm
- net +12V_MCU: track 200.4 -> 226.0 mm
- net +16V_INV: track 126.1 -> 128.9 mm
- net +24V_MCU: track 53.5 -> 51.8 mm
- net +3V3_MCU: track 17.1 -> 16.1 mm
- net Net-(U3-VFB): track 2.99 -> 3.53 mm
- added copper zone on B.Cu, net +12V_MCU
- added copper zone on F.Cu, net +12V_MCU
- added copper zone on In1.Cu, net +12V_MCU
- added copper zone on In2.Cu, net +12V_MCU
- added copper zone on B.Cu, net +16V_INV
- added copper zone on B.Cu, net +24V_INV
- added copper zone on F.Cu, net +24V_INV
- added copper zone on In1.Cu, net +24V_INV
- added copper zone on B.Cu, net +24V_MCU
- added copper zone on F.Cu, net +24V_MCU
- added copper zone on B.Cu, net +3V3_MCU
- added copper zone on B.Cu, net +5V_INV
- added copper zone on B.Cu, net +5V_MCU
- added copper zone on B.Cu, net GND_INV
- added copper zone on F.Cu, net GND_INV
- added copper zone on In1.Cu, net GND_INV
- added copper zone on In2.Cu, net GND_INV
- added copper zone on B.Cu, net GND_MCU
- added copper zone on F.Cu, net GND_MCU
- added copper zone on In1.Cu, net GND_MCU
- added copper zone on In2.Cu, net GND_MCU
- added copper zone on B.Cu, net Net-(RL1-COIL1)
- added copper zone on B.Cu, net Net-(RL2-COIL2)
- added copper zone on B.Cu, net Net-(U1-SW)
- added copper zone on B.Cu, net Net-(U3-SW)

Commit message: V1 layout update 4
Routing:
- net Net-(C8-Pad1): track 35.4 -> 49.2 mm
- net CHASSIS: track 158.2 -> 168.2 mm, vias 1 -> 11
- net Net-(C11-Pad1): track 37.4 -> 39.9 mm
- net Net-(RL2-NC): track 142.1 -> 140.1 mm
- net PGND: track 173.6 -> 175.2 mm
- net Net-(G1-Pad2): track 18.5 -> 19.4 mm
- added copper zone on B.Cu, net CHASSIS
- added copper zone on F.Cu, net CHASSIS
- added copper zone on In1.Cu, net CHASSIS
- added copper zone on In2.Cu, net CHASSIS
- added copper zone on B.Cu, net Net-(G1-Pad2)
- added copper zone on B.Cu, net PGND
- added copper zone on F.Cu, net PGND
- added copper zone on In1.Cu, net PGND
- added copper zone on In2.Cu, net PGND
- added copper zone on B.Cu, net VDC
- added copper zone on F.Cu, net VDC
- added copper zone on In1.Cu, net VDC
- added copper zone on In2.Cu, net VDC

Commit message: V1 layout update 5
Routing:
- net CHASSIS: track 168.2 -> 257.6 mm, vias 11 -> 14
Changed lines of the file:
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@@
 		(pad_to_mask_clearance 0)
 		(allow_soldermask_bridges_in_footprints no)
-		(grid_origin 92.3375 67.205)
+		(grid_origin 117.2375 54.855)
 		(pcbplotparams
 			(layerselection 0x00010fc_ffffffff)
@@
 	)
 	(gr_line
+		(start 85.9875 68.554565)
+		(end 103.3375 68.554565)
+		(stroke
+			(width 1.2)
+			(type default)
+		)
+		(layer "B.Mask")
+	)
+	(gr_line
+		(start 103.336739 68.554565)
+		(end 120.0375 51.853804)
+		(stroke
+			(width 1.2)
+			(type default)
+		)
+		(layer "B.Mask")
+	)
+	(gr_line
 		(start 138.8375 129.655)
 		(end 159.8375 108.655)
@@
 	)
 	(gr_line
+		(start 85.9875 65.855)
+		(end 85.9875 68.555)
+		(stroke
+			(width 1.2)
+			(type default)
+		)
+		(layer "B.Mask")
+	)
+	(gr_line
 		(start 145.7875 131.655)
 		(end 148.0875 129.355)
@@
 	(gr_line
 		(start 169.7375 61.855)
-		(end 162.7375 54.855)
+		(end 159.73679 51.85429)
 		(stroke
 			(width 1.2)
@@
 	)
 	(gr_line
-		(start 127.2375 54.855)
-		(end 162.7375 54.855)
+		(start 120.0375 51.853804)
+		(end 159.7375 51.853804)
 		(stroke
 			(width 1.2)
@@
 	)
 	(gr_line
+		(start 85.9875 65.855)
+		(end 102.1375 65.855)
+		(stroke
+			(width 1.2)
+			(type default)
+		)
+		(layer "B.Mask")
+	)
+	(gr_line
+		(start 102.1375 65.855)
+		(end 118.13627 49.85623)
+		(stroke
+			(width 1.2)
+			(type default)
+		)
+		(layer "B.Mask")
+	)
+	(gr_line
 		(start 159.8375 108.655)
 		(end 159.8375 103.655)
@@
 	(segment
 		(start 92.3375 67.205)
-		(end 92.3375 80.355)
-		(width 0.16)
+		(end 92.3375 77.355)
+		(width 0.5)
 		(layer "F.Cu")
 		(net 18)
@@
 	)
 	(segment
-		(start 92.3375 80.355)
+		(start 89.3375 80.355)
+		(end 84.5875 80.355)
+		(width 0.5)
+		(layer "F.Cu")
+		(net 18)
+	)
+	(segment
+		(start 95.3375 80.355)
 		(end 100.0875 80.355)
-		(width 0.16)
+		(width 0.5)
 		(layer "F.Cu")
 		(net 18)
@@
 		(start 168.7375 55.614999)
 		(end 168.7375 58.155)
-		(width 0.16)
-		(layer "F.Cu")
-		(net 18)
-	)
-	(segment
-		(start 100.0875 80.355)
-		(end 84.5875 80.355)
-		(width 0.16)
+		(width 1)
 		(layer "F.Cu")
 		(net 18)
@@
 	)
 	(via
+		(at 166.5875 55.614999)
+		(size 0.48)
+		(drill 0.3)
+		(layers "F.Cu" "B.Cu")
+		(net 18)
+	)
+	(via
 		(at 91.3375 67.205)
 		(size 0.48)
@@
 	)
 	(via
+		(at 165.5875 55.614999)
+		(size 0.48)
+		(drill 0.3)
+		(layers "F.Cu" "B.Cu")
+		(net 18)
+	)
+	(via
+		(at 166.5875 56.614999)
+		(size 0.48)
+		(drill 0.3)
+		(layers "F.Cu" "B.Cu")
+		(net 18)
+	)
+	(via
 		(at 90.3375 67.205)
 		(size 0.48)
@@
 		(net 18)
 	)
+	(arc
+		(start 92.3375 77.355)
+		(mid 91.45882 79.47632)
+		(end 89.3375 80.355)
+		(width 0.5)
+		(layer "F.Cu")
+		(net 18)
+	)
+	(arc
+		(start 95.3375 80.355)
+		(mid 93.21618 79.47632)
+		(end 92.3375 77.355)
+		(width 0.5)
+		(layer "F.Cu")
+		(net 18)
+	)
 	(segment
-		(start 92.3375 59.305)
-		(end 92.3375 51.615)
-		(width 0.16)
-		(layer "B.Cu")
+		(start 165.5875 55.614999)
+		(end 166.5875 55.614999)
+		(width 1)
+		(layer "In2.Cu")
 		(net 18)
 	)
 	(segment
-		(start 166.197499 55.614999)
+		(start 165.5875 55.614999)
+		(end 166.5875 56.614999)
+		(width 1)
+		(layer "In2.Cu")
+		(net 18)
+	)
+	(segment
+		(start 102.7375 67.205)
+		(end 119.5875 50.355)
+		(width 1)
+		(layer "In2.Cu")
+		(net 18)
+	)
+	(segment
+		(start 166.5875 55.614999)
 		(end 168.7375 55.614999)
 		(width 1)
-		(layer "B.Cu")
+		(layer "In2.Cu")
 		(net 18)
 	)
 	(segment
-		(start 116.737501 51.805)
-		(end 162.3875 51.805)
+		(start 163.2125 53.239999)
+		(end 164.452501 54.48)
 		(width 1)
-		(layer "B.Cu")
+		(layer "In2.Cu")
 		(net 18)
 	)
 	(segment
 		(start 87.3375 67.205)
-		(end 95.3375 67.205)
+		(end 102.7375 67.205)
 		(width 1)
+		(layer "In2.Cu")
+		(net 18)
+	)
+	(segment
+		(start 166.5875 56.614999)
+		(end 168.127501 58.155)
+		(width 1)
+		(layer "In2.Cu")
+		(net 18)
+	)
+	(segment
+		(start 168.127501 58.155)
+		(end 168.7375 58.155)
+		(width 1)
+		(layer "In2.Cu")
+		(net 18)
+	)
+	(segment
+		(start 119.5875 50.355)
+		(end 160.327501 50.355)
+		(width 1)
+		(layer "In2.Cu")
+		(net 18)
+	)
+	(segment
+		(start 163.2125 53.239999)
+		(end 165.5875 55.614999)
+		(width 1)
+		(layer "In2.Cu")
+		(net 18)
+	)
+	(segment
+		(start 160.327501 50.355)
+		(end 163.2125 53.239999)
+		(width 1)
+		(layer "In2.Cu")
+		(net 18)
+	)
+	(segment
+		(start 97.3375 67.205)
+		(end 102.7375 67.205)
+		(width 1)
+		(layer "B.Cu")
+		(net 18)
+	)
+	(segment
+		(start 160.3375 50.355)
+		(end 165.5875 55.605)
+		(width 1)
+		(layer "B.Cu")
+		(net 18)
+	)
+	(segment
+		(start 92.3375 59.305)
+		(end 92.3375 51.615)
+		(width 0.16)
 		(layer "B.Cu")
 		(net 18)
 	)
 	(segment
-		(start 162.3875 51.805)
-		(end 165.4625 54.88)
+		(start 168.432501 58.46)
+		(end 165.5875 55.614999)
 		(width 1)
 		(layer "B.Cu")
@@
 	)
 	(segment
-		(start 165.4625 54.88)
-		(end 166.197499 55.614999)
+		(start 119.5875 50.355)
+		(end 160.3375 50.355)
 		(width 1)
 		(layer "B.Cu")
@@
 	)
 	(segment
-		(start 97.3375 67.205)
-		(end 101.337501 67.205)
+		(start 102.7375 67.205)
+		(end 119.5875 50.355)
 		(width 1)
 		(layer "B.Cu")
@@
 	)
 	(segment
-		(start 95.3375 67.205)
-		(end 96.3375 67.205)
+		(start 87.3375 67.205)
+		(end 95.3375 67.205)
 		(width 1)
 		(layer "B.Cu")
@@
 	)
 	(segment
-		(start 165.4625 54.88)
+		(start 168.7375 55.614999)
 		(end 168.7375 58.155)
 		(width 1)
@@
 	)
 	(segment
-		(start 101.337501 67.205)
-		(end 116.737501 51.805)
+		(start 168.7375 58.155)
+		(end 168.432501 58.46)
+		(width 1)
+		(layer "B.Cu")
+		(net 18)
+	)
+	(segment
+		(start 95.3375 67.205)
+		(end 96.3375 67.205)
+		(width 1)
+		(layer "B.Cu")
+		(net 18)
+	)
+	(segment
+		(start 165.5875 55.605)
+		(end 165.5875 55.614999)
 		(width 1)
 		(layer "B.Cu")
@@
 		(polygon
 			(pts
-				(xy 85.6875 69.155) (xy 87.3875 69.155) (xy 88.4375 68.105) (xy 96.2375 68.105) (xy 97.2875 69.155)
-				(xy 98.9875 69.155) (xy 98.9875 68.105) (xy 93.8375 62.955) (xy 93.8375 50.365) (xy 90.8375 50.365)
-				(xy 90.8375 62.955) (xy 85.6875 68.105)
+				(xy 85.6875 69.155) (xy 87.3875 69.155) (xy 88.4375 68.105) (xy 91.3375 68.105) (xy 92.3375 69.105)
+				(xy 93.3375 68.105) (xy 96.2375 68.105) (xy 97.2875 69.155) (xy 98.9875 69.155) (xy 98.9875 68.105)
+				(xy 93.8375 62.955) (xy 93.8375 50.365) (xy 90.8375 50.365) (xy 90.8375 62.955) (xy 85.6875 68.105)
 			)
 		)
@@
 			)
 		)
+	)
+	(zone
+		(net 18)
+		(net_name "CHASSIS")
+		(layers "F.Cu" "In1.Cu" "In2.Cu" "B.Cu")
+		(hatch edge 0.5)
+		(priority 7)
+		(connect_pads yes
+			(clearance 0)
+		)
+		(min_thickness 0.25)
+		(filled_areas_thickness no)
+		(fill yes
+			(thermal_gap 0.25)
+			(thermal_bridge_width 0.25)
+		)
+		(polygon
+			(pts
+				(xy 169.3875 54.714999) (xy 169.6375 54.955) (xy 169.6375 56.635) (xy 169.6375 58.555) (xy 169.1375 59.055)
+				(xy 168.3375 59.055) (xy 163.997499 54.714999) (xy 163.997499 54.714999) (xy 167.2875 54.714999)
+			)
+		)

Commit message: HW.ACIM-PSU_REV1.0 production
Parts:
- added G***: LOGO, LOGO, F.Cu at (164.2, 50.4)
- added G***: LOGO, LOGO, F.Cu at (73.6, 86.5)
- added G***: LOGO, LOGO, F.Cu at (114.0, 50.4)
- added G***: LOGO, LOGO, F.Cu at (112.4, 135.0)
- added G***: LOGO, LOGO, F.Cu at (168.1, 86.7)
- added G***: LOGO, LOGO, F.Cu at (106.2, 90.5)
- added G***: LOGO, LOGO, F.Cu at (73.5, 55.3)
- added G***: LOGO, LOGO, F.Cu at (78.4, 145.5)
- added G***: LOGO, LOGO, F.Cu at (166.9, 141.3)
Routing:
- net CHASSIS: track 257.6 -> 476.7 mm, vias 14 -> 33
- net PGND: track 175.2 -> 31.8 mm, vias 0 -> 92
- net Net-(RL2-NC): track 140.1 -> 0.00 mm, vias 0 -> 73
- net Net-(MD2-ACL): track 51.2 -> 159.3 mm
- net Net-(MD1-ACL): track 33.9 -> 126.7 mm
- net Net-(MD2-ACN): track 60.5 -> 131.6 mm
- net Net-(MD1-ACN): track 23.9 -> 94.4 mm
- net AC1: track 40.3 -> 95.7 mm
- net AC2: track 33.6 -> 78.5 mm
- net Net-(BR1-DC+): track 21.7 -> 0.00 mm, vias 0 -> 28
- net +12V_MCU: track 226.0 -> 228.0 mm
- net +24V_INV: track 32.7 -> 34.3 mm
- net VDC: vias 0 -> 40
- net Net-(C8-Pad1): vias 0 -> 7
- net Net-(C11-Pad1): vias 0 -> 13
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- added copper zone on F.Cu, net +16V_INV
- added copper zone on In1.Cu, net +16V_INV
- added copper zone on In2.Cu, net +16V_INV
- added copper zone on B.Cu, net AC1
- added copper zone on F.Cu, net AC1
- added copper zone on In1.Cu, net AC1
- added copper zone on In2.Cu, net AC1
- added copper zone on B.Cu, net AC2
- added copper zone on F.Cu, net AC2
- added copper zone on In1.Cu, net AC2
- added copper zone on In2.Cu, net AC2
- added copper zone on B.Cu, net Net-(BR1-DC+)
- added copper zone on F.Cu, net Net-(BR1-DC+)
- added copper zone on In1.Cu, net Net-(BR1-DC+)
- added copper zone on In2.Cu, net Net-(BR1-DC+)
- added copper zone on B.Cu, net Net-(C11-Pad1)
- added copper zone on F.Cu, net Net-(C11-Pad1)
- added copper zone on In1.Cu, net Net-(C11-Pad1)
- added copper zone on In2.Cu, net Net-(C11-Pad1)
- added copper zone on B.Cu, net Net-(C8-Pad1)
- added copper zone on F.Cu, net Net-(C8-Pad1)
- added copper zone on In1.Cu, net Net-(C8-Pad1)
- added copper zone on In2.Cu, net Net-(C8-Pad1)
- added copper zone on B.Cu, net Net-(R4-Pad1)
- added copper zone on B.Cu, net Net-(RL2-NC)
- added copper zone on F.Cu, net Net-(RL2-NC)
- added copper zone on In1.Cu, net Net-(RL2-NC)
- added copper zone on In2.Cu, net Net-(RL2-NC)
Other:
- board text added: "CHASSIS"
- board text added: "HW.ACIM-PSU V1.0"
- board text added: "PGND"
- board text added: "SAFE-ZONE"
- board text added: "VDC"
