File: Design/HW.ACIM-PSU/HW.ACIM-PSU.kicad_sch (KiCad schematic)
At the start: 8 parts

Commit message: V1 layout update 1
Parts:
- added SH9: SCREW HOLDER, SAMPI:SCREWHOLE-2.5M, symbol SAMPI:SCREWHOLDER
Changed lines of the file:
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@@
+	(symbol
+		(lib_id "SAMPI:SCREWHOLDER")
+		(at 82.55 86.995 0)
+		(unit 1)
+		(exclude_from_sim no)
+		(in_bom yes)
+		(on_board yes)
+		(dnp no)
+		(property "Reference" "SH9"
+			(at 81.28 86.995 0)
+			(effects
+				(font
+					(face "Consolas")
+					(size 1.27 1.27)
+					(thickness 0.254)
+					(bold yes)
+				)
+				(justify left)
+			)
+		)
+		(property "Value" "SCREW HOLDER"
+			(at 85.09 92.0749 0)
+			(effects
+				(font
+					(face "Consolas")
+					(size 1.016 1.016)
+					(thickness 0.127)
+				)
+				(justify left)
+				(hide yes)
+			)
+		)
+		(property "Footprint" "SAMPI:SCREWHOLE-2.5M"
+			(at 82.55 86.995 0)
+			(effects
+				(font
+					(face "Consolas")
+					(size 1.016 1.016)
+					(thickness 0.127)
+				)
+				(hide yes)
+			)
+		)
+		(property "Datasheet" ""
+			(at 82.55 86.995 0)
+			(effects
+				(font
+					(face "Consolas")
+					(size 1.016 1.016)
+					(thickness 0.127)
+				)
+				(hide yes)
+			)
+		)
+		(property "Description" "PAN PHILLIPS SCREW, M2.5 X 4.5 T"
+			(at 82.55 86.995 0)
+			(effects
+				(font
+					(face "Consolas")
+					(size 1.016 1.016)
+					(thickness 0.127)
+				)
+				(hide yes)
+			)
+		)
+		(property "MFT" "Essentra"
+			(at 82.55 86.995 0)
+			(effects
+				(font
+					(face "Consolas")
+					(size 1.016 1.016)
+				)
+				(hide yes)
+			)
+		)
+		(property "MNP" "50M025045P012"
+			(at 82.55 86.995 0)
+			(effects
+				(font
+					(face "Consolas")
+					(size 1.016 1.016)
+				)
+				(hide yes)
+			)
+		)
+		(instances
+			(project "HW.ACIM-PSU"
+				(path "/20f80521-75f2-4ccc-bb34-c9566e70ef5c"
+					(reference "SH9")
+					(unit 1)
+				)
+			)
+		)
+	)
 	(symbol
 		(lib_id "SAMPI:SCREWHOLDER")

Commit message: HW.ACIM-PSU_REV1.0 production
Other:
- note removed: "Inter-Connection"
Changed lines of the file:
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@@
-		)
-	)
-	(text "Inter-Connection"
-		(exclude_from_sim no)
-		(at 211.455 163.83 0)
-		(effects
-			(font
-				(face "Consolas")
-				(size 1.016 1.016)
-				(thickness 0.127)
-			)
 		)
 	)
