File: Design/HW.ACIM-PSU/INVPOWER.kicad_sch (KiCad schematic)
At the start: 55 parts, among them J1 POWER CONN, J2 LINE, J3 INV PWR & RELAYS, J4 HIGH VOLTAGE OUTPUTS, J7 TE, J8 NEUTRAL, M1 470V/1.2kA, M2 470V/1.2kA, M3 470V/1.2kA, Q1 20V/1A, Q2 20V/1A, U1 SMPS 16V±2%/0.6A, U2 LDO 5V±1%

Commit message: V1 layout
Connections:
- net PGND: now also J4.10, J4.8, J4.9; no longer J4.4, J4.5, J4.6
- net VDC: now also J4.4, J4.5, J4.6; no longer J4.10, J4.8, J4.9
- net at C6.1, FT1.4: now also MD1.2 (ACL); no longer MD1.1 (ACN)
- net at C6.2, FT1.2: now also MD1.1 (ACN); no longer MD1.2 (ACL)
Other:
- moved on the sheet: B1, BR1, C1, C10, C11, C12, C13, C14, C15, C16, C2, C3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

Commit message: V1 layout update 1
Parts:
- added C31: 10uF/35V, SAMPI:CAP1206, symbol SAMPI:CERCAP
- added D7: PWR, SAMPI:LED0603, symbol SAMPI:WLED
- added R15: 1K, SAMPI:RES0603, symbol SAMPI:RES
- C10: value 470uF/25V -> 220uF/25V; footprint SAMPI:CAP_ELEC-10.3x10.3-DIA10 -> SAMPI:CAP_ELEC-8.3x8.3-DIA8.0; MFT KEMET -> Panasonic; MNP A768MS477M1ELAE017 -> EEH-ZL1E221XP
Connections:
- net +12V_MCU: now also RL2.1 (COIL1); no longer RL2.2 (COIL2)
- net +16V_INV: now also C31.2
- net +5V_INV: now also D7.A
- net GND_INV: now also C31.1, R15.2
- net PWR_RELAY: now also J3.7; no longer J3.8
- net ~{DEV_RELAY}: now also J3.8; no longer J3.7
- net at D4.K, D5.A: now also RL2.2 (COIL2); no longer RL2.1 (COIL1)
- new net: D7.K, R15.1
Other:
- moved on the sheet: C12, U2
